Commit message: now we use xacro format, and execute join_states for use robot tfs

File: blue_description/urdf/blue.xacro (robot description, xacro)
@@ -1,52 +1,7 @@
 <?xml version="1.0"?>
 <robot name="blue" xmlns:xacro="http://www.ros.org/wiki/xacro">
-  <material name="black">
-    <color rgba="0.0 0.0 0.0 1.0"/>
-  </material>
-  <material name="blue">
-    <color rgba="0.203125 0.23828125 0.28515625 1.0"/>
-  </material>
-  <material name="green">
-    <color rgba="0.0 0.8 0.0 1.0"/>
-  </material>
-  <material name="grey">
-    <color rgba="0.2 0.2 0.2 1.0"/>
-  </material>
-  <material name="orange">
-    <color rgba="1.0 0.423529411765 0.0392156862745 1.0"/>
-  </material>
-  <material name="brown">
-    <color rgba="0.870588235294 0.811764705882 0.764705882353 1.0"/>
-  </material>
-  <material name="red">
-    <color rgba="0.80078125 0.12890625 0.1328125 1.0"/>
-  </material>
-  <material name="white">
-    <color rgba="1.0 1.0 1.0 1.0"/>
-  </material>
-  <gazebo reference="link_chassis">
-    <material>Gazebo/Orange</material>
-  </gazebo>
-  <gazebo reference="link_left_wheel">
-    <material>Gazebo/Blue</material>
-  </gazebo>
-  <gazebo reference="link_right_wheel">
-    <material>Gazebo/Blue</material>
-  </gazebo>
-  <gazebo>
-    <plugin filename="libgazebo_ros_diff_drive.so" name="differential_drive_controller">
-      <alwaysOn>true</alwaysOn>
-      <updateRate>20</updateRate>
-      <leftJoint>joint_left_wheel</leftJoint>
-      <rightJoint>joint_right_wheel</rightJoint>
-      <wheelSeparation>0.4</wheelSeparation>
-      <wheelDiameter>0.2</wheelDiameter>
-      <torque>0.1</torque>
-      <commandTopic>cmd_vel</commandTopic>
-      <odometryTopic>odom</odometryTopic>
-      <odometryFrame>odom</odometryFrame>
-      <robotBaseFrame>link_chassis</robotBaseFrame>
-    </plugin>
-  </gazebo>
+  <xacro:include filename="$(find blue_description)/urdf/blue_materials.xacro" />
+  <xacro:include filename="$(find blue_description)/urdf/blue.gazebo" />
+  <xacro:include filename="$(find blue_description)/urdf/macros.xacro" />
   <link name="link_chassis">
     <!-- pose and inertial -->
@@ -92,62 +47,8 @@
       </geometry>
     </visual>
-    </link>
-  <!-- Create wheel right -->
-  <link name="link_right_wheel">
-    <inertial>
-      <mass value="0.2"/>
-      <origin rpy="0 1.5707 1.5707" xyz="0 0 0"/>
-      <inertia ixx="0.00052666666" ixy="0" ixz="0" iyy="0.00052666666" iyz="0" izz="0.001"/>
-    </inertial>
-    <collision name="link_right_wheel_collision">
-      <origin rpy="0 1.5707 1.5707" xyz="0 0 0" />
-      <geometry>
-        <cylinder length="0.04" radius="0.1"/>
-      </geometry>
-    </collision>
-    <visual name="link_right_wheel_visual">
-      <origin rpy="0 1.5707 1.5707" xyz="0 0 0"/>
-      <geometry>
-        <cylinder length="0.04" radius="0.1"/>
-      </geometry>
-    </visual>
   </link>
-  <!--   Joint for right wheel  -->
-  <joint name="joint_right_wheel" type="continuous">
-    <origin rpy="0 0 0" xyz="-0.05 0.15 0"/>
-    <child link="link_right_wheel" />
-    <parent link="link_chassis"/>
-    <axis rpy="0 0 0" xyz="0 1 0"/>
-    <limit effort="10000" velocity="1000"/>
-    <joint_properties damping="1.0" friction="1.0" />
-  </joint>
-  <!-- Left Wheel link -->
-  <link name="link_left_wheel">
-    <inertial>
-      <mass value="0.2"/>
-      <origin rpy="0 1.5707 1.5707" xyz="0 0 0"/>
-      <inertia ixx="0.00052666666" ixy="0" ixz="0" iyy="0.00052666666" iyz="0" izz="0.001"/>
-    </inertial>
-    <collision name="link_left_wheel_collision">
-      <origin rpy="0 1.5707 1.5707" xyz="0 0 0" />
-      <geometry>
-        <cylinder length="0.04" radius="0.1"/>
-      </geometry>
-    </collision>
-    <visual name="link_left_wheel_visual">
-      <origin rpy="0 1.5707 1.5707" xyz="0 0 0"/>
-      <geometry>
-        <cylinder length="0.04" radius="0.1"/>
-      </geometry>
-    </visual>
-  </link>
-  <!--   Joint for right wheel  -->
-  <joint name="joint_left_wheel" type="continuous">
-    <origin rpy="0 0 0" xyz="-0.05 -0.15 0"/>
-    <child link="link_left_wheel" />
-    <parent link="link_chassis"/>
-    <axis rpy="0 0 0" xyz="0 1 0"/>
-    <limit effort="10000" velocity="1000"/>
-    <joint_properties damping="1.0" friction="1.0" />
-  </joint>
+  <xacro:link_wheel name="link_right_wheel" />
+  <xacro:join_wheel name="joint_right_wheel" child="link_right_wheel" origin_xyz="-0.05 0.15 0"/>
+  <xacro:link_wheel name="link_left_wheel" />
+  <xacro:join_wheel name="joint_left_wheel" child="link_left_wheel" origin_xyz="-0.05 -0.15 0"/>
 </robot>

Commit message: modifications in gazebo model to simulate tricicle model

File: blue_description/urdf/blue.xacro (robot description, xacro)
@@ -4,51 +4,14 @@
   <xacro:include filename="$(find blue_description)/urdf/blue.gazebo" />
   <xacro:include filename="$(find blue_description)/urdf/macros.xacro" />
-  <link name="link_chassis">
-    <!-- pose and inertial -->
-    <pose>0 0 0.1 0 0 0</pose>
-    <inertial>
-      <mass value="5"/>
-      <origin rpy="0 0 0" xyz="0 0 0.1"/>
-      <inertia ixx="0.0395416666667" ixy="0" ixz="0" iyy="0.106208333333" iyz="0" izz="0.106208333333"/>
-    </inertial>
-    <collision name="collision_chassis">
-      <geometry>
-        <box size="0.5 0.3 0.07"/>
-      </geometry>
-    </collision>
-    <visual>
-      <origin rpy="0 0 0" xyz="0 0 0"/>
-      <geometry>
-        <box size="0.5 0.3 0.07"/>
-      </geometry>
-      <material name="blue"/>
-    </visual>
-    <!-- caster front -->
-    <collision name="caster_front_collision">
-      <origin rpy=" 0 0 0" xyz="0.35 0 -0.05"/>
-      <geometry>
-        <sphere radius="0.05"/>
-      </geometry>
-      <surface>
-        <friction>
-          <ode>
-            <mu>0</mu>
-            <mu2>0</mu2>
-            <slip1>1.0</slip1>
-            <slip2>1.0</slip2>
-          </ode>
-        </friction>
-      </surface>
-    </collision>
-    <visual name="caster_front_visual">
-      <origin rpy=" 0 0 0" xyz="0.2 0 -0.05"/>
-      <geometry>
-        <sphere radius="0.05"/>
-      </geometry>
-    </visual>
-  </link>
-  <xacro:link_wheel name="link_right_wheel" />
-  <xacro:join_wheel name="joint_right_wheel" child="link_right_wheel" origin_xyz="-0.05 0.15 0"/>
-  <xacro:link_wheel name="link_left_wheel" />
-  <xacro:join_wheel name="joint_left_wheel" child="link_left_wheel" origin_xyz="-0.05 -0.15 0"/>
+  <xacro:base name="base_link" />
+  <xacro:caster name="caster_link" />
+  <xacro:caster_join name="front_caster_join" child="caster_link" origin_xyz="0.6 0 -0.203"/>
+  <xacro:wheel name="front_right_wheel_link" length="0.12" radius="0.18" />
+  <xacro:wheel_join name="front_right_wheel_join" child="front_right_wheel_link" origin_xyz="0.6 0.28 -0.203"/>
+  <xacro:wheel name="front_left_wheel_link" length="0.12" radius="0.18" />
+  <xacro:wheel_join name="front_left_wheel_join" child="front_left_wheel_link" origin_xyz="0.6 -0.28 -0.203"/>
+  <xacro:wheel name="rear_right_wheel_link" length="0.18" radius="0.203" />
+  <xacro:wheel_join name="rear_right_wheel_link_join" child="rear_right_wheel_link" origin_xyz="-0.45 0.31 -0.203"/>
+  <xacro:wheel name="rear_left_wheel_link" length="0.18" radius="0.203" />
+  <xacro:wheel_join name="rear_left_wheel_link_join" child="rear_left_wheel_link" origin_xyz="-0.45 -0.31 -0.203"/>
 </robot>

File: blue_description/urdf/macros.xacro (robot description, xacro)
@@ -1,5 +1,25 @@
 <?xml version="1.0"?>
 <robot>
-  <macro name="link_wheel" params="name">
+  <macro name="base" params="name">
+    <link name="${name}">
+      <inertial>
+        <mass value="5"/>
+        <origin rpy="0 0 0" xyz="-0.45 0 -0.203"/>
+        <inertia ixx="0.0395416666667" ixy="0" ixz="0" iyy="0.106208333333" iyz="0" izz="0.106208333333"/>
+      </inertial>
+      <collision name="${name}_collision">
+        <geometry>
+          <box size="1.672 0.797 0.03"/>
+        </geometry>
+      </collision>
+      <visual name="${name}_visual">
+        <geometry>
+          <box size="1.672 0.797 0.03"/>
+        </geometry>
+        <material name="blue"/>
+      </visual>
+    </link>
+  </macro>
+  <macro name="wheel" params="name length radius">
     <link name="${name}">
       <inertial>
@@ -11,5 +31,5 @@
         <origin rpy="0 1.5707 1.5707" xyz="0 0 0" />
         <geometry>
-         <cylinder length="0.04" radius="0.1"/>
+         <cylinder length="${length}" radius="${radius}"/>
         </geometry>
       </collision>
@@ -17,14 +37,15 @@
         <origin rpy="0 1.5707 1.5707" xyz="0 0 0"/>
         <geometry>
-          <cylinder length="0.04" radius="0.1"/>
+          <cylinder length="${length}" radius="${radius}"/>
         </geometry>
+        <material name="grey"/>
       </visual>
     </link>
   </macro>
-  <macro name="join_wheel" params="name child origin_xyz">
+  <macro name="wheel_join" params="name child origin_xyz">
       <joint name="${name}" type="continuous">
         <origin rpy="0 0 0" xyz="${origin_xyz}"/>
         <child link="${child}" />
-        <parent link="link_chassis"/>
+        <parent link="base_link"/>
         <axis rpy="0 0 0" xyz="0 1 0"/>
         <limit effort="10000" velocity="1000"/>
@@ -32,3 +53,25 @@
     </joint>
   </macro>
+  <macro name="caster" params="name">
+    <link name="${name}">
+      <inertial>
+        <mass value="3"/>
+        <origin rpy="0 0 0" xyz="0 0 0"/>
+        <inertia ixx="0" ixy="0" ixz="0" iyy="0" iyz="0" izz="0"/>
+      </inertial>
+      <collision name="caster_front_collision">
+        <origin rpy="0 1.5707 1.5707" xyz="0 0 0" />
+          <geometry>
+            <sphere radius="0.203"/>
+          </geometry>
+      </collision>
+    </link>
+  </macro>
+  <macro name="caster_join" params="name child origin_xyz">
+      <joint name="${name}" type="continuous">
+        <origin rpy="0 0 0" xyz="${origin_xyz}"/>
+        <child link="${child}" />
+        <parent link="base_link"/>
+    </joint>
+  </macro>
 </robot>

Commit message: velodyne simulation added to blue xacro model

File: blue_description/urdf/blue.xacro (robot description, xacro)
@@ -6,5 +6,7 @@
   <xacro:base name="base_link" />
   <xacro:caster name="caster_link" />
-  <xacro:caster_join name="front_caster_join" child="caster_link" origin_xyz="0.6 0 -0.203"/>
+  <xacro:generic_join name="front_caster_join" child="caster_link" origin_xyz="0.6 0 -0.203"/>
+  <xacro:bar name="lidar_bar_link" />
+  <xacro:generic_join name="lidar_bar_join" child="lidar_bar_link" origin_xyz="0 0 0.2"/>
   <xacro:wheel name="front_right_wheel_link" length="0.12" radius="0.18" />
   <xacro:wheel_join name="front_right_wheel_join" child="front_right_wheel_link" origin_xyz="0.6 0.28 -0.203"/>
@@ -15,3 +17,7 @@
   <xacro:wheel name="rear_left_wheel_link" length="0.18" radius="0.203" />
   <xacro:wheel_join name="rear_left_wheel_link_join" child="rear_left_wheel_link" origin_xyz="-0.45 -0.31 -0.203"/>
+  <xacro:include filename="$(find velodyne_description)/urdf/VLP-16.urdf.xacro"/>
+  <xacro:VLP-16 parent="base_link" name="velodyne" topic="/velodyne_points" hz="10" samples="440">
+    <origin xyz="0 0 0.4" rpy="0 0 0" />
+  </xacro:VLP-16>
 </robot>

File: blue_description/urdf/macros.xacro (robot description, xacro)
@@ -60,5 +60,5 @@
         <inertia ixx="0" ixy="0" ixz="0" iyy="0" iyz="0" izz="0"/>
       </inertial>
-      <collision name="caster_front_collision">
+      <collision name="${name}_collision">
         <origin rpy="0 1.5707 1.5707" xyz="0 0 0" />
           <geometry>
@@ -68,5 +68,27 @@
     </link>
   </macro>
-  <macro name="caster_join" params="name child origin_xyz">
+  <macro name="bar" params="name">
+    <link name="${name}">
+      <inertial>
+        <mass value="0.1"/>
+        <origin rpy="0 0 0" xyz="0 0 0"/>
+        <inertia ixx="0" ixy="0" ixz="0" iyy="0" iyz="0" izz="0"/>
+      </inertial>
+      <collision name="${name}_collision">
+        <origin rpy="0 0 0" xyz="0 0 0" />
+          <geometry>
+            <cylinder length="0.4" radius="0.02"/>
+          </geometry>
+      </collision>
+      <visual name="${name}_visual">
+        <origin rpy="0 0 0" xyz="0 0 0"/>
+        <geometry>
+          <cylinder length="0.4" radius="0.02"/>
+        </geometry>
+        <material name="white"/>
+      </visual>
+    </link>
+  </macro>
+  <macro name="generic_join" params="name child origin_xyz">
       <joint name="${name}" type="continuous">
         <origin rpy="0 0 0" xyz="${origin_xyz}"/>

Commit message: urban and robot modifications

File: blue_description/urdf/blue.xacro (robot description, xacro)
@@ -5,15 +5,17 @@
   <xacro:include filename="$(find blue_description)/urdf/macros.xacro" />
   <xacro:base name="base_link" />
+  <!--
   <xacro:caster name="caster_link" />
-  <xacro:generic_join name="front_caster_join" child="caster_link" origin_xyz="0.6 0 -0.203"/>
+  <xacro:generic_join name="front_caster_join" child="caster_link" origin_xyz="0 0 0"/>
+  -->
   <xacro:bar name="lidar_bar_link" />
   <xacro:generic_join name="lidar_bar_join" child="lidar_bar_link" origin_xyz="0 0 0.2"/>
-  <xacro:wheel name="front_right_wheel_link" length="0.12" radius="0.18" />
+  <xacro:wheel name="front_right_wheel_link" length="0.1" radius="0.18" />
   <xacro:wheel_join name="front_right_wheel_join" child="front_right_wheel_link" origin_xyz="0.6 0.28 -0.203"/>
-  <xacro:wheel name="front_left_wheel_link" length="0.12" radius="0.18" />
+  <xacro:wheel name="front_left_wheel_link" length="0.1" radius="0.18" />
   <xacro:wheel_join name="front_left_wheel_join" child="front_left_wheel_link" origin_xyz="0.6 -0.28 -0.203"/>
-  <xacro:wheel name="rear_right_wheel_link" length="0.18" radius="0.203" />
+  <xacro:wheel name="rear_right_wheel_link" length="0.12" radius="0.203" />
   <xacro:wheel_join name="rear_right_wheel_link_join" child="rear_right_wheel_link" origin_xyz="-0.45 0.31 -0.203"/>
-  <xacro:wheel name="rear_left_wheel_link" length="0.18" radius="0.203" />
+  <xacro:wheel name="rear_left_wheel_link" length="0.12" radius="0.203" />
   <xacro:wheel_join name="rear_left_wheel_link_join" child="rear_left_wheel_link" origin_xyz="-0.45 -0.31 -0.203"/>
   <xacro:include filename="$(find velodyne_description)/urdf/VLP-16.urdf.xacro"/>

File: blue_description/urdf/macros.xacro (robot description, xacro)
@@ -3,42 +3,60 @@
   <macro name="base" params="name">
     <link name="${name}">
-      <inertial>
-        <mass value="5"/>
-        <origin rpy="0 0 0" xyz="-0.45 0 -0.203"/>
-        <inertia ixx="0.0395416666667" ixy="0" ixz="0" iyy="0.106208333333" iyz="0" izz="0.106208333333"/>
-      </inertial>
-      <collision name="${name}_collision">
-        <geometry>
-          <box size="1.672 0.797 0.03"/>
-        </geometry>
-      </collision>
-      <visual name="${name}_visual">
-        <geometry>
-          <box size="1.672 0.797 0.03"/>
-        </geometry>
-        <material name="blue"/>
-      </visual>
+    <!-- pose and inertial -->
+    <pose>-0.45 0 -0.203 0 0 0</pose>
+    <inertial>
+      <mass value="5"/>
+      <origin rpy="0 0 0" xyz="-0.45 0 -0.203"/>
+      <inertia ixx="0.0395416666667" ixy="0" ixz="0" iyy="0.106208333333" iyz="0" izz="0.106208333333"/>
+    </inertial>
+    <collision name="${name}_collision">
+      <geometry>
+        <box size="1.672 0.797 0.03"/>
+      </geometry>
+    </collision>
+    <visual name="${name}_visual">
+      <origin rpy="0 0 0" xyz="0 0 0"/>
+      <geometry>
+        <box size="1.672 0.797 0.03"/>
+      </geometry>
+      <material name="blue"/>
+    </visual>
+    <collision name="${name}_caster_collision">
+      <origin rpy=" 0 0 0" xyz="0.6 0 -0.203"/>
+      <geometry>
+        <sphere radius="0.203"/>
+      </geometry>
+      <surface>
+        <friction>
+          <ode>
+            <mu>0</mu>
+            <mu2>0</mu2>
+            <slip1>1.0</slip1>
+            <slip2>1.0</slip2>
+          </ode>
+        </friction>
+      </surface>
+    </collision>
     </link>
   </macro>
   <macro name="wheel" params="name length radius">
     <link name="${name}">
-      <inertial>
-        <mass value="0.2"/>
-        <origin rpy="0 1.5707 1.5707" xyz="0 0 0"/>
-        <inertia ixx="0.00052666666" ixy="0" ixz="0" iyy="0.00052666666" iyz="0" izz="0.001"/>
-      </inertial>
-      <collision name="${name}_collision">
-        <origin rpy="0 1.5707 1.5707" xyz="0 0 0" />
-        <geometry>
-         <cylinder length="${length}" radius="${radius}"/>
-        </geometry>
-      </collision>
-      <visual name="${name}_visual">
-        <origin rpy="0 1.5707 1.5707" xyz="0 0 0"/>
-        <geometry>
-          <cylinder length="${length}" radius="${radius}"/>
-        </geometry>
-        <material name="grey"/>
-      </visual>
+    <inertial>
+      <mass value="0.2"/>
+      <origin rpy="0 1.5707 1.5707" xyz="0 0 0"/>
+      <inertia ixx="0.00052666666" ixy="0" ixz="0" iyy="0.00052666666" iyz="0" izz="0.001"/>
+    </inertial>
+    <collision name="${name}_collision">
+      <origin rpy="0 1.5707 1.5707" xyz="0 0 0" />
+      <geometry>
+        <cylinder length="${length}" radius="${radius}"/>
+      </geometry>
+    </collision>
+    <visual name="${name}_visual">
+      <origin rpy="0 1.5707 1.5707" xyz="0 0 0"/>
+      <geometry>
+        <cylinder length="${length}" radius="${radius}"/>
+      </geometry>
+    </visual>
     </link>
   </macro>
@@ -56,5 +74,5 @@
     <link name="${name}">
       <inertial>
-        <mass value="3"/>
+        <mass value="0.1"/>
         <origin rpy="0 0 0" xyz="0 0 0"/>
         <inertia ixx="0" ixy="0" ixz="0" iyy="0" iyz="0" izz="0"/>
@@ -62,7 +80,17 @@
       <collision name="${name}_collision">
         <origin rpy="0 1.5707 1.5707" xyz="0 0 0" />
-          <geometry>
-            <sphere radius="0.203"/>
-          </geometry>
+        <geometry>
+          <sphere radius="0.203"/>
+        </geometry>
+        <surface>
+          <friction>
+            <ode>
+              <mu>0</mu>
+              <mu2>0</mu2>
+              <slip1>1.0</slip1>
+              <slip2>1.0</slip2>
+            </ode>
+          </friction>
+        </surface>
       </collision>
     </link>
