Commit message: GPS join added to xacro.

File: blue_description/urdf/blue_ackerman.xacro (robot description, xacro)
@@ -75,9 +75,12 @@
   <xacro:property name="servo_stall_torque" value="5.649"/>
   <xacro:property name="servo_no_load_speed" value="4.553"/>
-  <material name="blue">
+   <material name="blue">
      <color rgba="0 0 0.8 1"/>
    </material>
    <material name="gray">
     <color rgba="0.5 0.5 0.5 1.0"/>
+   </material>
+      <material name="white">
+    <color rgba="1.0 1.0 1.0 1.0"/>
    </material>
    <material name="flat_black">
@@ -109,4 +112,22 @@
        rviz. -->
   <link name="base_link"/>
+  <joint name="gps_joint" type="fixed">
+    <parent link="base_link"/>
+    <child link="gps"/>
+    <origin xyz="0.82 -0.25 0.445" rpy="0.0 0.0 0.0"/>
+  </joint>
+  <link name='gps'>
+    <visual>
+      <geometry>
+        <cylinder length="0.05" radius="0.07"/>
+      </geometry>
+      <material name="white"/>
+    </visual>
+    <collision>
+      <geometry>
+        <cylinder length="0.05" radius="0.07"/>
+      </geometry>
+    </collision>
+  </link>
   <joint name="base_link_to_chassis" type="fixed">
     <parent link="base_link"/>
@@ -536,5 +557,5 @@
       <alwaysOn>true</alwaysOn>
       <updateRate>1.0</updateRate>
-      <bodyName>base_link</bodyName>
+      <bodyName>gps</bodyName>
       <topicName>fix</topicName>
       <velocityTopicName>fix_vel</velocityTopicName>
